Commit message: Change value of Length0

File: rrp_description/urdf/rrp.xacro (robot description, xacro)
@@ -4,5 +4,5 @@
   <!-- Constants for robot dimensions -->
   <xacro:property name="PI" value="3.1415926535897931"/>
-  <xacro:property name="length0" value="0.1" /> <!-- Base -->
+  <xacro:property name="length0" value="0.05" /> <!-- Base -->
   <xacro:property name="length1" value="0.45" /> <!-- Link 0 -->
   <xacro:property name="length2" value="0.425" /> <!-- Link 1 -->

Commit message: Updated base link length in xacro

File: rrp_description/urdf/rrp.xacro (robot description, xacro)
@@ -19,5 +19,5 @@
     <visual>
       <geometry>
-        <box size = "0.2 ${length0} 0.05"/>
+        <box size = "0.2 0.1 ${length0}"/>
       </geometry>
       <material name = "white"/>
@@ -31,5 +31,5 @@
     <collision>
       <geometry>
-        <box size = "0.2 ${length0} 0.05"/>
+        <box size = "0.2 0.1 ${length0}"/>
       </geometry>
       <material name = "white"/>
